Commit message: add some

File: robots/kobuki_hexagons_hokuyo.urdf.xacro (robot description, xacro)
@@ -11,8 +11,7 @@
   <xacro:include filename="$(find mbot_gazebo)/urdf/kobuki.urdf.xacro" />
   <xacro:kobuki/>
-P
  <xacro:include filename="$(find mbot_gazebo)/urdf/stacks/circles.urdf.xacro"/>
   <xacro:include filename="$(find mbot_gazebo)/urdf/stacks/hexagons.urdf.xacro"/>
-  <xacro:include filename="$(find mbot_gazebo)/urdf/sensors/kinect.urdf.xacro"/>
+ <!-- <xacro:include filename="$(find mbot_gazebo)/urdf/sensors/kinect.urdf.xacro"/>-->
   <xacro:include filename="$(find mbot_gazebo)/urdf/sensors/hokuyo.urdf.xacro"/>
   <!--

File: urdf/create.urdf.xacro (robot description, xacro)
@@ -86,7 +86,7 @@
 	  </link>
 	  <joint name="base_footprint_joint" type="fixed">
-	    <origin xyz="0 0 0.017" rpy="0 0 0" />
-	    <parent link="base_footprint"/>
-	    <child link="base_link" />
+	    <origin xyz="0 0 -0.017" rpy="0 0 0" />
+	    <parent link="base_link"/>
+	    <child link="base_footprint" />
 	  </joint>
 	  <joint name="base_wall_sensor_joint" type="fixed">
